File: C64-Mouse-Adapter.kicad_pcb (KiCad board)
At the start: 2 copper layers, 42.9 x 16.9 mm, 12 parts, among them J1 AVR-ISP-6, J2 Joystick Port, J3 PS/2 Socket, SW1 RESET, U1 ATmega8-16AU

Commit message: Fixed DRC Problems
Routing:
- net Net-(R6-Pad2): track 14.9 -> 15.6 mm
- net GND: vias 27 -> 21
Other:
- board text added: "Rev 2 ~PCB: baldenginer.com Circuit: sensi.org/~~svo/[m]ouse"
- board text removed: "Rev 1 ~PCB: baldenginer.com Circuit: sensi.org/~~svo/[m]ouse"
